File: PCB (schematics + pcb)/Luma pcb.kicad_sch (KiCad schematic)
At the start: 20 parts, among them J1 Conn_01x04_Pin, SW1 SW_Push, SW2 SW_Push, SW3 SW_Push, SW4 SW_Push, SW5 SW_Push, SW6 RotaryEncoder_Switch, U1 MOUDLE-SEEEDUINO-XIAO

Commit message: Add QMK firmware matching PCB netlist, CAD case files, and PCB updates
Firmware (XIAO RP2040):
- Add keyboard.json with correct pins traced from the PCB netlist:
  switches on GP26/GP27/GP28/GP29/GP4, encoder on GP0/GP1 with push
  button on GP2, OLED I2C on GP6/GP7, 5x SK6812 RGB LEDs on GP3
- Fix keymap.c: invalid X_LSHIFT keycode, KC_NO interception replaced
  with a proper ANIM_CYCLE keycode, encoder push mapped to mute
- Add three animated OLED modes (scanner, equalizer, breathing logo)
  with a live last-action status line
- Enable RGBLIGHT for the onboard LED chain

Also add CAD case STEP files and gitignore editor auto-backups.

Co-Authored-By: Claude Fable 5 <noreply@anthropic.com>
Parts:
- D1, D2, D3, D4, D5: value WS2812B -> SK6812MINI-E; footprint LED_SMD:LED_WS2812B_PLCC4_5.0x5.0mm_P3.2mm -> footprints:SK6812MINI-E_fixed
Other:
- moved on the sheet: D4
Changed lines of the file:
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@@
 	)
 	(junction
-		(at 176.784 111.252)
+		(at 208.026 45.974)
 		(diameter 0)
 		(color 0 0 0 0)
 	)
 	(junction
-		(at 273.05 43.688)
+		(at 176.784 111.252)
 		(diameter 0)
 		(color 0 0 0 0)
 	)
 	(junction
-		(at 208.026 45.974)
+		(at 273.05 43.688)
 		(diameter 0)
 		(color 0 0 0 0)
@@
 	)
 	(junction
-		(at 220.726 38.354)
+		(at 158.496 92.456)
 		(diameter 0)
 		(color 0 0 0 0)
 	)
 	(junction
-		(at 158.496 92.456)
+		(at 56.388 118.872)
 		(diameter 0)
 		(color 0 0 0 0)
 	)
 	(junction
-		(at 56.388 118.872)
+		(at 161.798 79.502)
 		(diameter 0)
 		(color 0 0 0 0)
 	)
 	(junction
-		(at 161.798 79.502)
+		(at 220.726 37.338)
 		(diameter 0)
 		(color 0 0 0 0)
@@
 	(wire
 		(pts
+			(xy 220.726 37.338) (xy 220.726 38.354)
+		)
+		(stroke
+			(width 0)
+			(type default)
+		)
+	)
+	(wire
+		(pts
 			(xy 149.86 118.364) (xy 149.86 147.066)
 		)
@@
 	(wire
 		(pts
-			(xy 215.646 38.354) (xy 220.726 38.354)
+			(xy 215.138 37.338) (xy 220.726 37.338)
 		)
 		(stroke
@@
 	(wire
 		(pts
+			(xy 207.518 44.958) (xy 208.026 45.974)
+		)
+		(stroke
+			(width 0)
+			(type default)
+		)
+	)
+	(wire
+		(pts
 			(xy 169.926 84.582) (xy 169.926 76.708)
 		)
@@
 	(wire
 		(pts
+			(xy 215.138 52.578) (xy 215.646 53.594)
+		)
+		(stroke
+			(width 0)
+			(type default)
+		)
+	)
+	(wire
+		(pts
 			(xy 155.956 95.504) (xy 155.956 93.98)
 		)
@@
 	(wire
 		(pts
-			(xy 220.726 22.86) (xy 220.726 38.354)
+			(xy 220.726 22.86) (xy 220.726 37.338)
 		)
 		(stroke
@@
 	(wire
 		(pts
-			(xy 242.824 45.974) (xy 223.266 45.974)
+			(xy 242.824 44.958) (xy 222.758 44.958)
 		)
 		(stroke
@@
 	(wire
 		(pts
-			(xy 242.824 39.878) (xy 242.824 45.974)
+			(xy 242.824 39.878) (xy 242.824 44.958)
 		)
 		(stroke
@@
 			)
 		)
-		(property "Value" "WS2812B"
+		(property "Value" "SK6812MINI-E"
 			(at 156.718 40.64 0)
 			(show_name no)
@@
 			)
 		)
-		(property "Footprint" "LED_SMD:LED_WS2812B_PLCC4_5.0x5.0mm_P3.2mm"
+		(property "Footprint" "footprints:SK6812MINI-E_fixed"
 			(at 176.784 52.07 0)
 			(hide yes)
@@
 			)
 		)
-		(property "Value" "WS2812B"
+		(property "Value" "SK6812MINI-E"
 			(at 280.924 47.4278 0)
 			(show_name no)
@@
 			)
 		)
-		(property "Footprint" "LED_SMD:LED_WS2812B_PLCC4_5.0x5.0mm_P3.2mm"
+		(property "Footprint" "footprints:SK6812MINI-E_fixed"
 			(at 271.78 58.928 0)
 			(hide yes)
@@
 			)
 		)
-		(property "Value" "WS2812B"
+		(property "Value" "SK6812MINI-E"
 			(at 264.16 34.9818 0)
 			(show_name no)
@@
 			)
 		)
-		(property "Footprint" "LED_SMD:LED_WS2812B_PLCC4_5.0x5.0mm_P3.2mm"
+		(property "Footprint" "footprints:SK6812MINI-E_fixed"
 			(at 254 63.5 0)
 			(hide yes)
@@
 	(symbol
 		(lib_id "LED:WS2812B")
-		(at 215.646 45.974 0)
+		(at 215.138 44.958 0)
 		(unit 1)
 		(body_style 1)
@@
 		(dnp no)
 		(property "Reference" "D4"
-			(at 250.444 42.6018 0)
+			(at 249.936 41.5858 0)
 			(show_name no)
 			(do_not_autoplace no)
@@
 			)
 		)
-		(property "Value" "WS2812B"
-			(at 226.06 42.0938 0)
+		(property "Value" "SK6812MINI-E"
+			(at 225.552 41.0778 0)
 			(show_name no)
 			(do_not_autoplace no)
@@
 			)
 		)
-		(property "Footprint" "LED_SMD:LED_WS2812B_PLCC4_5.0x5.0mm_P3.2mm"
-			(at 216.916 53.594 0)
+		(property "Footprint" "footprints:SK6812MINI-E_fixed"
+			(at 216.408 52.578 0)
 			(hide yes)
 			(show_name no)
@@
 		)
 		(property "Datasheet" "https://cdn-shop.adafruit.com/datasheets/WS2812B.pdf"
-			(at 218.186 55.499 0)
+			(at 217.678 54.483 0)
 			(hide yes)
 			(show_name no)
@@
 		)
 		(property "Description" "RGB LED with integrated controller"
-			(at 215.646 45.974 0)
+			(at 215.138 44.958 0)
 			(hide yes)
 			(show_name no)
@@
 			)
 		)
-		(property "Value" "WS2812B"
+		(property "Value" "SK6812MINI-E"
 			(at 117.348 55.2606 0)
 			(show_name no)
@@
 			)
 		)
-		(property "Footprint" "LED_SMD:LED_WS2812B_PLCC4_5.0x5.0mm_P3.2mm"
+		(property "Footprint" "footprints:SK6812MINI-E_fixed"
 			(at 105.664 50.546 0)
 			(hide yes)
