File: PCB (schematics + pcb)/Luma pcb.kicad_pcb (KiCad board)
At the start: 2 copper layers, 77.6 x 78.3 mm, 22 parts, among them J1 Conn_01x04_Pin, SW1 SW_Push, SW2 SW_Push, SW3 SW_Push, SW4 SW_Push, SW5 SW_Push, SW6 RotaryEncoder_Switch, U1 MOUDLE-SEEEDUINO-XIAO

Commit message: added small changes to pcb
Parts:
- added G***: LOGO, LOGO, F.Cu at (130.2, 124.5)
- moved G*** 14.6 mm to (147.4, 104.2)
